File: Arc_Reactor_PCB.kicad_pcb (KiCad board)
At the start: 4 copper layers, 70 x 70 mm, 42 parts, among them J1 Conn_01x01, J2 Conn_01x01, J3 USB_C_Receptacle, J4 Conn_01x03, SW1 SW_Push, SW2 SW_Push, U1 ESP32-C3-MINI-1, U2 AP63205WU, U3 SN74AHCT1G125, U4 LM66200DRLR, U5 AP2112K-3.3

Commit message: Improve WIFI Antenna Keepout
Parts:
- moved L1 1.10 mm to (105.7, 113.6)
- moved D1 0.65 mm to (105.2, 117.9)
- moved C4 0.50 mm to (102.2, 113.3)
- moved C7 0.50 mm to (99.2, 117.1)
- moved U2 0.50 mm to (99.2, 114.3)
Routing:
- net GND: track 14.9 -> 13.0 mm, vias 244 -> 253
- net BUCK_5V: track 27.2 -> 26.5 mm
Other:
- board text added: "BOOT"
- board text added: "RST"
